File: hardware/musiq-player-hardware/musiq-player-hardware.kicad_pcb (KiCad board)
At the start: 2 copper layers, 40.3 x 75.7 mm, 64 parts, among them J1 Micro_SD_Card, J2 AudioJack3, J3 TP4056_CONN, J4 UART, SW1 SW_MEC_5E, SW2 SW_MEC_5E, SW3 SW_MEC_5E, SW4 SW_MEC_5E, SW5 SW_MEC_5E, SW6 RST, SW8 ON/OFF, U1 74LVC125, U2 W25Q128JVS, U4 AMS1117-3.3, U5 ESP32C3, U6 MAX98357AETE, Y1 40MHz

Commit message: adds final PCB renders
Parts:
- renumbered J2 to AUD, SW3 to DOWN, SW4 to LEFT, SW1 to MENU, J1 to MICRO-SD, SW5 to RIGHT, SW6 to RST, J4 to UART, SW2 to UP
Other:
- board text added: "3V3"
- board text added: "4V2"
- board text added: "GND"
- board text added: "OFF"
- board text added: "ON"
- board text added: "PLAYA v1"
- board text added: "RX0"
- board text added: "SCL"
- board text added: "SDA"
- board text added: "TX0"
- board text added: "VCC"

Commit message: adds final PCB renders
Parts:
- moved AUD 0.16 mm to (139.3, 93.0)
Other:
- board size 40.3 x 75.7 mm -> 40.3 x 75.6 mm
Changed lines of the file:
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@@
   )
   (footprint "Connector_Audio:Jack_3.5mm_CUI_SJ1-3525N_Horizontal" (layer "F.Cu")
-    (at 139.33 93.21)
+    (at 139.29 93.05)
     (descr "TRS 3.5mm, horizontal, through-hole, https://www.cuidevices.com/product/resource/pdf/sj1-352xn.pdf")
     (tags "TRS audio jack stereo horizontal")
@@
         (effects (font (size 1 1) (thickness 0.15)))
     )
-    (fp_text user "PCB edge" (at 0 3.65 unlocked) (layer "Dwgs.User")
+    (fp_text user "PCB edge" (at 7.06 0.71 unlocked) (layer "Dwgs.User") hide
         (effects (font (size 1 1) (thickness 0.15)))
     )
@@
   (gr_line (start 152.61 47.31) (end 154.2 47.31)
     (stroke (width 0.15) (type default)) (layer "F.SilkS"))
-  (gr_rect (start 118.295 21.91) (end 158.595 97.62)
-    (stroke (width 0.1) (type default)) (fill none) (layer "Edge.Cuts"))
+  (gr_line (start 158.59 21.92) (end 118.29 21.93)
+    (stroke (width 0.1) (type default)) (layer "Edge.Cuts"))
+  (gr_line (start 118.3 97.57) (end 132.67 97.57)
+    (stroke (width 0.1) (type default)) (layer "Edge.Cuts"))
+  (gr_line (start 132.79 97.57) (end 132.79 97.55)
+    (stroke (width 0.1) (type default)) (layer "Edge.Cuts"))
+  (gr_line (start 132.67 97.57) (end 132.79 97.57)
+    (stroke (width 0.1) (type default)) (layer "Edge.Cuts"))
+  (gr_line (start 145.97 97.55) (end 158.56 97.55)
+    (stroke (width 0.1) (type default)) (layer "Edge.Cuts"))
+  (gr_line (start 158.56 97.55) (end 158.59 21.92)
+    (stroke (width 0.1) (type default)) (layer "Edge.Cuts"))
+  (gr_line (start 118.29 21.93) (end 118.3 97.57)
+    (stroke (width 0.1) (type default)) (layer "Edge.Cuts"))
+  (gr_line (start 145.97 97.55) (end 145.79 97.55)
+    (stroke (width 0.1) (type default)) (layer "Edge.Cuts"))
   (gr_text "VCC\n" (at 153.48 48.16) (layer "F.Cu")
     (effects (font (size 0.7 1) (thickness 0.175) bold) (justify left bottom))

Commit message: adds 3D design files
Parts:
- moved H3 47.9 mm to (163.0, 142.2)
- moved R1 47.9 mm to (149.1, 122.3)
- moved C1 47.9 mm to (143.7, 122.3)
- moved C10 47.9 mm to (133.8, 133.4)
- moved D1 47.9 mm to (138.5, 133.4)
- moved H1 47.9 mm to (128.5, 71.8)
- moved LEFT 47.9 mm to (132.9, 116.7)
- moved MENU 47.9 mm to (145.6, 116.5)
- moved R11 47.9 mm to (137.3, 104.3)
- moved R12 47.9 mm to (138.4, 130.7)
- moved R13 47.9 mm to (161.4, 109.0)
- moved R16 47.9 mm to (132.6, 129.8)
- moved R18 47.9 mm to (132.7, 125.5)
- moved R19 47.9 mm to (132.7, 123.4)
- moved R6 47.9 mm to (159.3, 86.7)
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Other:
- board size 40.3 x 75.6 mm -> 40.3 x 75.7 mm
